Commit message: 完成了基础的moveit controller的编写,10.10/1.37

File: src/arm_config/config/arm.ros2_control.xacro (robot description, xacro)
@@ -2,5 +2,5 @@
 <robot xmlns:xacro="http://www.ros.org/wiki/xacro">
     <xacro:macro name="arm_ros2_control" params="name initial_positions_file">
-        <xacro:property name="initial_positions" value="${xacro.load_yaml(initial_positions_file)['initial_positions']}"/>
+        <xacro:property name="initial_positions" value="${load_yaml(initial_positions_file)['initial_positions']}"/>
         <ros2_control name="${name}" type="system">
             <hardware>

File: src/arm_description/urdf/arm.xacro (robot description, xacro)
@@ -2,5 +2,4 @@
 <robot name="arm" xmlns:xacro="http://www.ros.org/wiki/xacro">
 <xacro:include filename="$(find arm_description)/urdf/materials.xacro" />
-<xacro:include filename="$(find arm_description)/urdf/arm.ros2control" />
 <xacro:include filename="$(find arm_description)/urdf/arm.gazebo" />
 <link name="base_link">
